File: PCB/Phoenixia.kicad_pcb (KiCad board)
At the start: 2 copper layers, 333.8 x 105.2 mm, 207 parts, among them J2 Button, J5 Conn_01x03_Male, K0 Blank, K1 Blank, K10 Blank, K11 Blank, K12 Blank, K13 Blank, K14 Blank, K15 Blank, K16 Blank, K17 Blank, K18 Blank, K19 Blank, K2 Blank, K20 Blank, K21 Blank, K22 Blank, K23 Blank, K24 Blank, K25 Blank, K26 Blank, K27 Blank, K28 Blank, K29 Blank, K3 Blank, K30 Blank, K31 Blank, K32 Blank, K33 Blank, K34 Blank, K35 Blank, K36 Blank, K37 Blank, K38 Blank, K39 Blank, K4 Blank, K40 Blank, K41 Blank, K42 Blank, K43 Blank, K44 Blank, K45 Blank, K46 Blank, K47 Blank, K48 Blank, K49 Blank, K5 Blank, K50 Blank, K51 Blank, K52 Blank, K53 Blank, K54 Blank, K55 Blank, K56 Blank, K57 Blank, K58 Blank, K59 Blank, K6 Blank, K60 Blank, K61 Blank, K62 Blank, K63 Blank, K64 Blank, K65 Blank, K66 Blank, K67 Blank, K68 Blank, K69 Blank, K7 Blank, K70 Blank, K71 Blank, K72 Blank, K73 Blank, K74 Blank, K75 Blank, K76 Blank, K8 Blank, K9 Blank, U1 SOT-23-5 5.5V 3.3V 500mA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

Commit message: Fixed Files
Parts:
- removed the C1 at (356.5, 83.9)
- removed C20: 100nf 0402, Capacitor_SMD:C_0402_1005Metric
- removed MX_SK6812MINI-E: MX_SK6812MINI-E, kicad-keyboard-parts:MX_SK6812MINI-E
- removed the U3 at (356.9, 82.0)
- D0, D1, D10, D11, D12, D13, D14, D15, D16, D17, D18, D19, D2, D20, D21, D22, D23, D24, D25, D26, D27, D28, D29, D3, D30, D31, D32, D33, D34, D35, D36, D37, D38, D39, D4, D40, D41, D42, D43, D44, D45, D46, D47, D48, D49, D5, D50, D51, D52, D53, D54, D55, D56, D57, D58, D59, D6, D60, D61, D62, D63, D64, D65, D66, D67, D68, D69, D7, D70, D71, D72, D73, D74, D75, D76, D8, D9: footprint Diode_SMD:D_SOD-123 -> Diode_SMD:D_SOD-123F
- D100: renamed from D1; value 1N4002W -> schottky
- DLED1: renamed from D2; footprint LED_SMD:LED_0402_1005Metric -> Diode_SMD:D_0402_1005Metric
- K0, K1, K10, K11, K12, K13, K14, K15, K16, K17, K18, K19, K2, K20, K21, K22, K23, K24, K25, K26, K27, K28, K29, K3, K30, K31, K32, K33, K34, K35, K36, K37, K38, K39, K4, K40, K41, K42, K43, K44, K45, K46, K47, K48, K49, K5, K50, K51, K52, K53, K54, K55, K56, K57, K58, K59, K6, K60, K61, K62, K63, K64, K65, K66, K67, K68, K69, K7, K70, K71, K72, K73, K74, K75, K76, K8, K9: footprint Button_Switch_Keyboard:SW_Cherry_Choc4_MX_1.00u_PCB -> Button_Switch_Keyboard:SW_Cherry_Choc3_MX_1.00u_PCB
- R9: value 1k -> 62ohm 0402
- moved D74 0.68 mm to (319.3, 109.3)
- moved D73 0.67 mm to (300.3, 109.3)
- moved D13 0.64 mm to (400.4, 47.1)
- moved D14 0.64 mm to (419.5, 47.1)
- moved D23 0.64 mm to (262.2, 64.9)
- moved D29 0.64 mm to (400.4, 66.2)
- moved D30 0.64 mm to (419.5, 66.2)
- moved D45 0.64 mm to (400.4, 85.2)
- moved D46 0.64 mm to (419.5, 85.2)
- moved D61 0.64 mm to (400.4, 104.2)
- moved D62 0.64 mm to (419.5, 104.2)
- moved D7 0.64 mm to (262.2, 45.9)
- moved D0 0.64 mm to (128.9, 45.8)
- moved D1 0.64 mm to (147.9, 45.9)
- moved D16 0.64 mm to (128.9, 64.9)
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Connections:
- net /Col_0 renamed Col_0
- net /Col_1 renamed Col_1
- net /Col_10 renamed Col_10
- net /Col_11 renamed Col_11
- net /Col_13 renamed Col_13
- net /Col_14 renamed Col_14
- net /Col_15 renamed Col_15
- net /Col_2 renamed Col_2
- net /Col_3 renamed Col_3
- net /Col_4 renamed Col_4
- net /Col_5 renamed Col_5
- net /Col_6 renamed Col_6
- net /Col_7 renamed Col_7
- net /Col_8 renamed Col_8
- net /Col_9 renamed Col_9
- net /Row3 renamed Row_3
- net /Row_0 renamed Row_0
- net /Row_1 renamed Row_1
- net /Row_2 renamed Row_2
- net /Row_4 renamed Row_4
- net SPARE8 renamed SPARE7
- net UNUSED renamed SPARE6
- DLED1 pad 1: LED_RES -> unconnected-(DLED1-K-Pad1)
- K12 pad 1: /Col_12 -> Col_12
- K28 pad 1: /Col_12 -> Col_12
- K44 pad 1: /Col_12 -> Col_12
- K60 pad 1: /Col_12 -> Col_12
- K76 pad 1: Net-(D76-A) -> Col_12
- K76 pad 2: /Col_12 -> Net-(D76-A)
- R9 pad 1: GND -> unconnected-(R9-Pad1)
- R9 pad 2: LED_RES -> unconnected-(R9-Pad2)
- U3 pad 18: /Col_12 -> Col_12
- U3 pad 27: MIDLED_SRC -> SPARE5
Routing:
- net Col_12: track 0.00 -> 155.1 mm, vias 0 -> 2
- net /Col_12: track 140.2 -> 0.00 mm, vias 2 -> 0
- net VSYS: track 85.3 -> 6.93 mm, vias 2 -> 1
- net +3V3: track 105.4 -> 63.7 mm, vias 6 -> 5
- net MIDLED_SRC: track 21.7 -> 0.00 mm
- net GND: track 42.8 -> 26.7 mm
- net Col_4: track 245.5 -> 260.0 mm
- net Col_0: track 322.7 -> 337.1 mm
- net Col_2: track 284.4 -> 298.5 mm
- net Col_1: track 303.5 -> 317.6 mm
- net Col_9: track 147.5 -> 161.6 mm
- net Col_10: track 128.3 -> 142.4 mm
- net Col_11: track 109.1 -> 123.2 mm
- net Col_3: track 265.2 -> 279.2 mm
- net Col_8: track 166.8 -> 180.7 mm
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