File: PCB/Phoenixia3.kicad_pcb (KiCad board)
At the start: 2 copper layers, 348.6 x 161.2 mm, 134 parts, among them K0 Blank, K1 Blank, K10 Blank, K11 Blank, K16 Blank, K17 Blank, K18 Blank, K19 Blank, K2 Blank, K20 Blank, K21 Blank, K22 Blank, K23 Blank, K24 Blank, K25 Blank, K26 Blank, K27 Blank, K3 Blank, K32 Blank, K33 Blank, K34 Blank, K35 Blank, K36 Blank, K37 Blank, K38 Blank, K39 Blank, K4 Blank, K40 Blank, K41 Blank, K42 Blank, K43 Blank, K44 Blank, K48 Blank, K49 Blank, K5 Blank, K50 Blank, K51 Blank, K52 Blank, K53 Blank, K54 Blank, K55 Blank, K56 Blank, K57 Blank, K58 Blank, K59 Blank, K6 Blank, K60 Blank, K64 Blank, K65 Blank, K66 Blank, K67 Blank, K68 Blank, K69 Blank, K7 Blank, K70 Blank, K71 Blank, K72 Blank, K73 Blank, K74 Blank, K75 Blank, K8 Blank, K9 Blank, U1 Pico

Commit message: Shape
Parts:
- added ?: , , F.Cu at (207.4, 163.3)
- added H4: MountingHole, MountingHole:MountingHole_2.2mm_M2_Pad, F.Cu at (65.6, 178.2)
- added H4: MountingHole, MountingHole:MountingHole_2.2mm_M2_Pad, F.Cu at (207.4, 234.7)
- added H4: MountingHole, MountingHole:MountingHole_2.2mm_M2_Pad, F.Cu at (105.4, 82.7)
- added H4: MountingHole, MountingHole:MountingHole_2.2mm_M2_Pad, F.Cu at (38.0, 131.0)
- added H4: MountingHole, MountingHole:MountingHole_2.2mm_M2_Pad, B.Cu at (376.8, 131.0)
- added H4: MountingHole, MountingHole:MountingHole_2.2mm_M2_Pad, B.Cu at (309.4, 82.7)
- added H4: MountingHole, MountingHole:MountingHole_2.2mm_M2_Pad, B.Cu at (349.2, 178.2)
- G***: moved to B.Cu
- K1, K10, K11, K2, K3, K4, K5, K6, K7, K8, K9: footprint Button_Switch_Keyboard:SW_Cherry_Choc5_MX_1.00u_PCB_LED -> Button_Switch_Keyboard:SW_Cherry_Choc5_MX_1.00u_PCB_LED_3D2
- K17, K18, K19, K20, K21, K22, K23, K24, K25, K26, K27, K32, K33, K34, K35, K36, K37, K38, K39, K40, K41, K42, K43, K44 (x2), K48, K49, K50, K51, K52, K53, K54, K55, K56, K57, K58, K59, K60 (x2), K64, K65, K66, K67, K68, K69 (x2), K70 (x2), K71, K72, K73, K74, K75: footprint Button_Switch_Keyboard:SW_Cherry_Choc5_MX_1.00u_PCB -> Button_Switch_Keyboard:SW_Cherry_Choc5_MX_1.00u_PCB_3D
- pico: renamed from U1; value Pico -> (none)
- moved D54 31.2 mm to (246.5, 165.1)
- moved D50 31.2 mm to (97.5, 144.6)
- moved D49 31.2 mm to (78.3, 142.5)
- moved D58 31.2 mm to (320.4, 146.9)
- moved D25 31.2 mm to (291.4, 112.1)
- moved K44 31.2 mm to (366.1, 128.5)
- moved D56 31.2 mm to (282.4, 152.3)
- moved K71 31.2 mm to (262.4, 182.8)
- moved K9 31.2 mm to (297.4, 92.9)
- moved D33 31.2 mm to (83.2, 124.2)
- moved D6 31.2 mm to (231.6, 109.8)
- moved D40 31.2 mm to (277.5, 133.9)
- moved D72 31.2 mm to (269.4, 177.1)
- moved D67 31.2 mm to (129.4, 172.8)
- moved D69 31.2 mm to (169.9, 186.2)
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Connections:
- D69 pad 2: Net-(D69-A) -> NET-(DEXT-A)
- K11 pad 2: LED13 -> Net-(D11-A)
- K69 pad 2: Net-(D69-A) -> NET-(DEXT-A)
- pico pad 10: Col_15 -> Col_5
- pico pad 11: Col_14 -> Row_1
- pico pad 12: Col_13 -> Row_2
- pico pad 14: Row_2 -> Row_3
- pico pad 15: Col_9 -> Row_4
- pico pad 16: Row_3 -> (no net)
- pico pad 17: Row_4 -> (no net)
- pico pad 19: Col_8 -> Col_6
- pico pad 20: UNUSED -> Col_7
- pico pad 21: Col_7 -> Col_8
- pico pad 22: Col_6 -> Col_9
- pico pad 25: UNUSED2 -> Col_10
- pico pad 26: Col_2 -> Col_11
- pico pad 27: Col_1 -> Col_12
- pico pad 29: Col_0 -> Col_13
- pico pad 31: Col_5 -> Col_14
- pico pad 32: Col_4 -> Col_15
- pico pad 34: Col_3 -> Row_0
- pico pad 4: Row_0 -> Col_0
- pico pad 5: Col_12 -> Col_1
- pico pad 6: Col_11 -> Col_2
- pico pad 7: Col_10 -> Col_3
- pico pad 9: Row_1 -> Col_4
Routing:
- net Col_15: track 0.00 -> 246.3 mm
- net Col_14: track 0.00 -> 219.9 mm
- net Row_4: track 324.2 -> 544.0 mm, vias 0 -> 1
- net Col_13: track 0.00 -> 205.0 mm
- net Col_12: track 0.00 -> 190.2 mm
- net Row_3: track 137.3 -> 319.3 mm, vias 0 -> 2
- net Col_11: track 0.00 -> 170.3 mm
- net Col_10: track 0.00 -> 154.0 mm
- net VBUS: track 247.9 -> 323.6 mm
- net Row_2: track 219.9 -> 292.0 mm, vias 0 -> 2
- net LED7: track 6.90 -> 74.8 mm, vias 0 -> 4
- net Col_8: track 2.99 -> 64.1 mm
- net Row_1: track 217.6 -> 278.5 mm, vias 0 -> 2
- net Row_0: track 216.9 -> 274.4 mm, vias 0 -> 2
- net Col_5: track 95.6 -> 129.1 mm
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Other:
- board text added: "01 | Pi Pico 66 | 1N4148W 66 | Switches 66 | 1U Keycaps 14 | SK6812 MINI-E"
- board text added: "Model: Ashwing66 - (Choc V1/MX) Designed by: James Gzowski (github.com/gzowski)"
- board text added: "Pico goes here."
