File: PCB/Ashwing66_baseplate.kicad_pcb (KiCad board)
At the start: 2 copper layers, 348.6 x 161.2 mm, 11 parts

Commit message: Change of DIODE
Parts:
- removed ?: , 
Changed lines of the file:
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@@
 		(grid_origin 202.173552 167.880917)
 		(pcbplotparams
-			(layerselection 0x00318ff_ffffffff)
+			(layerselection 0x00010ff_ffffffff)
 			(plot_on_all_layers_selection 0x0000000_00000000)
 			(disableapertmacros no)
@@
 			(drillshape 0)
 			(scaleselection 1)
-			(outputdirectory "Gerber/")
+			(outputdirectory "Gerber Files/Base Plate/")
 		)
 	)
 	(net 0 "")
 	(net 1 "GND")
-	(footprint ""
-		(layer "F.Cu")
-		(at 39.048552 191.880917 -15)
-		(property "Reference" ""
-			(at 0 0 -15)
-			(unlocked yes)
-			(layer "F.SilkS")
-			(effects
-				(font
-					(size 1.27 1.27)
-				)
-			)
-		)
-		(property "Value" ""
-			(at 0 0 -15)
-			(unlocked yes)
-			(layer "F.Fab")
-			(effects
-				(font
-					(size 1.27 1.27)
-				)
-			)
-		)
-		(property "Footprint" ""
-			(at 0 0 -15)
-			(unlocked yes)
-			(layer "F.Fab")
-			(hide yes)
-			(effects
-				(font
-					(size 1.27 1.27)
-				)
-			)
-		)
-		(property "Datasheet" ""
-			(at 0 0 -15)
-			(unlocked yes)
-			(layer "F.Fab")
-			(hide yes)
-			(effects
-				(font
-					(size 1.27 1.27)
-				)
-			)
-		)
-		(property "Description" ""
-			(at 0 0 -15)
-			(unlocked yes)
-			(layer "F.Fab")
-			(hide yes)
-			(effects
-				(font
-					(size 1.27 1.27)
-				)
-			)
-		)
-		(pad "" thru_hole circle
-			(at 0 0 345)
-			(size 4 4)
-			(drill 2.4)
-			(layers "*.Cu" "*.Mask")
-			(remove_unused_layers no)
-		)
-	)
 	(footprint "Stencils:HOLE_M2_TH_SCREW"
 		(layer "F.Cu")
