File: PCB/Ashwing66_baseplate.kicad_pcb (KiCad board)
At the start: 2 copper layers, 348.6 x 161.2 mm, 10 parts

Commit message: new layout, added RGB
Parts:
- removed TH3 (x10): HOLE, Stencils:HOLE_M2_TH_SCREW
Other:
- board size 348.6 x 161.2 mm -> 346.6 x 149.9 mm
- board text added: "${REFERENCE}"

Commit message: Updates
Routing:
- removed copper zone on B.Cu, net GND
- removed copper zone on F.Cu, net GND
Other:
- board text removed: "${REFERENCE}"
Changed lines of the file:
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@@
 			(sketchpadsonfab no)
 			(subtractmaskfromsilk yes)
-			(outputformat 1)
+			(outputformat 4)
 			(mirror no)
 			(drillshape 0)
 			(scaleselection 1)
-			(outputdirectory "Gerber Files/Base Plate/")
+			(outputdirectory "../../../../")
 		)
 	)
 	(net 0 "")
-	(net 1 "GND")
 	(gr_line
 		(start 113.579903 90.803638)
@@
 		(layer "Edge.Cuts")
 	)
-	(gr_text "${REFERENCE}"
-		(at 131.164026 139.233336 165)
-		(layer "F.Fab")
-		(effects
-			(font
-				(size 1 1)
-				(thickness 0.15)
-			)
-		)
-	)
-	(zone
-		(net 1)
-		(net_name "GND")
-		(layers "F&B.Cu")
-		(hatch edge 0.5)
-		(connect_pads
-			(clearance 0.25)
-		)
-		(min_thickness 0.25)
-		(filled_areas_thickness no)
-		(fill yes
-			(thermal_gap 0.5)
-			(thermal_bridge_width 0.5)
-		)
-		(polygon
-			(pts
-				(xy 57.963552 74.190917) (xy 348.943552 76.250917) (xy 386.543552 117.450917) (xy 389.113552 154.530917)
-				(xy 355.123552 213.750917) (xy 207.923552 265.250917) (xy 16.343552 173.060917) (xy 57.963552 74.700917)
-			)
-		)
-	)
 )
