File: PCB/Ashwing66_topplate.kicad_pcb (KiCad board)
At the start: 2 copper layers, 348.6 x 161.2 mm, 75 parts, among them K0 Blank, K1 Blank, K10 Blank, K11 Blank, K16 Blank, K17 Blank, K18 Blank, K19 Blank, K2 Blank, K20 Blank, K21 Blank, K22 Blank, K23 Blank, K24 Blank, K25 Blank, K26 Blank, K27 Blank, K3 Blank, K32 Blank, K33 Blank, K34 Blank, K35 Blank, K36 Blank, K37 Blank, K38 Blank, K39 Blank, K4 Blank, K40 Blank, K41 Blank, K42 Blank, K43 Blank, K44 Blank, K48 Blank, K49 Blank, K5 Blank, K50 Blank, K51 Blank, K52 Blank, K53 Blank, K54 Blank, K55 Blank, K56 Blank, K57 Blank, K58 Blank, K59 Blank, K6 Blank, K60 Blank, K64 Blank, K65 Blank, K66 Blank, K67 Blank, K68 Blank, K69 Blank, K7 Blank, K70 Blank, K71 Blank, K72 Blank, K73 Blank, K74 Blank, K75 Blank, K8 Blank, K9 Blank

Commit message: Sun Jun  2 02:56:42 AM BST 2024
Parts:
- removed G***: LOGO, LOGO
- removed H4 (x7): MountingHole, MountingHole:MountingHole_2.2mm_M2_Pad
- added TH3: HOLE, Stencils:HOLE_M2_TH_SCREW, F.Cu at (182.4, 191.4)
- added TH3: HOLE, Stencils:HOLE_M2_TH_SCREW, B.Cu at (272.8, 187.0)
- added TH3: HOLE, Stencils:HOLE_M2_TH_SCREW, F.Cu at (152.0, 186.9)
- added TH3: HOLE, Stencils:HOLE_M2_TH_SCREW, F.Cu at (166.8, 131.7)
- added TH3: HOLE, Stencils:HOLE_M2_TH_SCREW, F.Cu at (92.4, 114.8)
- added TH3: HOLE, Stencils:HOLE_M2_TH_SCREW, F.Cu at (77.6, 170.1)
- added TH3: HOLE, Stencils:HOLE_M2_TH_SCREW, B.Cu at (347.2, 170.1)
- added TH3: HOLE, Stencils:HOLE_M2_TH_SCREW, B.Cu at (258.0, 131.7)
- added TH3: HOLE, Stencils:HOLE_M2_TH_SCREW, B.Cu at (332.4, 114.9)
- added TH3: HOLE, Stencils:HOLE_M2_TH_SCREW, B.Cu at (242.4, 191.5)
- K0, K1, K10, K11, K16, K17, K18, K19, K2, K20, K21, K22, K23, K24, K25, K26, K27, K3, K32, K33, K34, K35, K36, K37, K38, K39, K4, K40, K41, K42, K43, K44 (x2), K48, K49, K5, K50, K51, K52, K53, K54, K55, K56, K57, K58, K59, K6, K60 (x2), K64, K65, K66, K67, K68, K69 (x2), K7, K70 (x2), K71, K72, K73, K74, K75, K8, K9: footprint Button_Switch_Keyboard:SW_Cherry_Choc5_MX_1.00u_PCB_LED_3D2_CUTOUT3 -> Button_Switch_Keyboard:SW_Cherry_Choc5_MX_1.00u_PCB_LED_3D2_CUTOUT_CLEAN
- moved ? 160.0 mm to (39.0, 191.9), turned to -15 degrees
- moved K8 16.9 mm to (283.7, 107.3)
- moved K25 16.9 mm to (307.4, 122.2)
- moved K60 16.9 mm to (188.1, 172.4)
- moved K7 16.9 mm to (265.7, 113.7)
- moved K58 16.9 mm to (336.5, 157.1)
- moved K53 16.9 mm to (167.3, 176.6)
- moved K41 16.9 mm to (312.4, 140.7)
- moved K66 16.9 mm to (126.3, 182.2)
- moved K52 16.9 mm to (149.3, 170.2)
- moved K26 16.9 mm to (326.6, 120.3)
- moved K57 16.9 mm to (317.3, 159.0)
- moved K55 16.9 mm to (280.5, 168.9)
- moved K49 16.9 mm to (93.2, 158.4)
- moved K5 16.9 mm to (182.1, 121.4)
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Other:
- outline, holes or cut-outs redrawn

Commit message: Change of DIODE
Parts:
- removed ?: , 
- added K60: Blank, Button_Switch_Keyboard:SW_Cherry_Choc5_MX_1.00u_PCB_LED_3D2_CUTOUT_CLEAN_Lines, F.Cu at (215.0, 186.8)
- K0, K1, K10, K11, K16, K17, K18, K19, K2, K20, K21, K22, K23, K24, K25, K26, K27, K3, K32, K33, K34, K35, K37, K38, K39, K4, K40, K41, K42, K43, K44 (x2), K48, K49, K5, K50, K51, K52, K53, K54, K55, K56, K57, K58, K59, K6, K60 (x2), K64, K65, K66, K67, K68, K69 (x2), K7, K70 (x2), K71, K72, K73, K74, K75, K8, K9: footprint Button_Switch_Keyboard:SW_Cherry_Choc5_MX_1.00u_PCB_LED_3D2_CUTOUT_CLEAN -> Button_Switch_Keyboard:SW_Cherry_Choc5_MX_1.00u_PCB_LED_3D2_CUTOUT_CLEAN_Lines
- K36: value Blank -> (none); footprint Button_Switch_Keyboard:SW_Cherry_Choc5_MX_1.00u_PCB_LED_3D2_CUTOUT_CLEAN -> Button_Switch_Keyboard:SW_Cherry_Choc5_MX_1.00u_PCB_LED_3D2_CUTOUT_CLEAN_Lines
