File: PCB/Ashwing66_topplate.kicad_pcb (KiCad board)
At the start: 2 copper layers, 348.6 x 161.2 mm, 77 parts, among them K0 Blank, K1 Blank, K10 Blank, K11 Blank, K16 Blank, K17 Blank, K18 Blank, K19 Blank, K2 Blank, K20 Blank, K21 Blank, K22 Blank, K23 Blank, K24 Blank, K25 Blank, K26 Blank, K27 Blank, K3 Blank, K32 Blank, K33 Blank, K34 Blank, K35 Blank, K37 Blank, K38 Blank, K39 Blank, K4 Blank, K40 Blank, K41 Blank, K42 Blank, K43 Blank, K44 Blank, K48 Blank, K49 Blank, K5 Blank, K50 Blank, K51 Blank, K52 Blank, K53 Blank, K54 Blank, K55 Blank, K56 Blank, K57 Blank, K58 Blank, K59 Blank, K6 Blank, K60 Blank, K64 Blank, K65 Blank, K66 Blank, K67 Blank, K68 Blank, K69 Blank, K7 Blank, K70 Blank, K71 Blank, K72 Blank, K73 Blank, K74 Blank, K75 Blank, K8 Blank, K9 Blank

Commit message: new layout, added RGB
Parts:
- removed TH3 (x10): HOLE, Stencils:HOLE_M2_TH_SCREW
- moved K33 4.83 mm to (94.7, 143.3)
- moved K39 4.83 mm to (272.1, 153.9)
- moved K67 4.83 mm to (140.8, 192.0)
- moved K9 4.83 mm to (299.0, 107.2)
- moved K36 4.83 mm to (150.7, 155.2)
- moved K55 4.83 mm to (277.0, 172.2)
- moved K70 4.83 mm to (242.6, 205.2)
- moved K38 4.83 mm to (254.1, 160.3)
- moved K41 4.83 mm to (308.9, 144.0)
- moved K58 4.83 mm to (333.0, 160.4)
- moved K70 4.83 mm to (224.0, 218.7)
- moved K1 4.83 mm to (104.6, 106.5)
- moved K11 4.83 mm to (337.0, 101.7)
- moved K5 4.83 mm to (178.6, 124.8)
- moved K60 4.83 mm to (55.0, 144.1)
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Other:
- board size 348.6 x 161.2 mm -> 346.6 x 149.9 mm

Commit message: Mon Jun 10 03:52:55 PM BST 2024-Final
Parts:
- moved K42 15.3 mm to (340.2, 132.6)
- moved K9 15.3 mm to (311.1, 97.8)
- moved K55 15.3 mm to (289.1, 162.9)
- moved K35 15.3 mm to (144.8, 139.4)
- moved K36 15.3 mm to (162.8, 145.8)
- moved K60 15.3 mm to (223.6, 180.7)
- moved K66 15.3 mm to (134.9, 176.2)
- moved K69 15.3 mm to (191.8, 198.3)
- moved K70 15.3 mm to (254.7, 195.8)
- moved K20 15.3 mm to (167.8, 127.4)
- moved K0 15.3 mm to (97.9, 93.7)
- moved K1 15.3 mm to (116.7, 97.1)
- moved K17 15.3 mm to (111.7, 115.5)
- moved K33 15.3 mm to (106.8, 133.9)
- moved K48 15.3 mm to (83.1, 148.9)
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Other:
- outline, holes or cut-outs redrawn

Commit message: Updates
Parts:
- removed the K60 at (223.6, 180.7)
- K0, K1, K10, K11, K16, K17, K18, K19, K2, K20, K21, K22, K23, K24, K25, K26, K27, K3, K32, K33, K34, K35, K36, K37, K38, K39, K4, K40, K41, K42, K43, K44 (x2), K48, K49, K5, K50, K51, K52, K53, K54, K55, K56, K57, K58, K59, K6, K60 (x2), K64, K65, K66, K67, K68, K69 (x2), K7, K70 (x2), K71, K72, K73, K74, K75, K8, K9: footprint Button_Switch_Keyboard:SW_Cherry_Choc5_MX_1.00u_PCB_LED_3D2_CUTOUT_CLEAN_Lines -> Button_Switch_Keyboard:SW_Cherry_Choc5_MX_1.00u_PCB_LED_3D2_CUTOUT_CLEAN_Lines_1.0
Routing:
- removed copper zone on B.Cu, net GND
- removed copper zone on F.Cu, net GND
Other:
- outline, holes or cut-outs redrawn
