File: PCB/Ashwing66_hard.kicad_pcb (KiCad board)
At the start: 2 copper layers, 346.6 x 149.9 mm, 148 parts, among them K0 Blank, K1 Blank, K10 Blank, K11 Blank, K16 Blank, K17 Blank, K18 Blank, K19 Blank, K2 Blank, K20 Blank, K21 Blank, K22 Blank, K23 Blank, K24 Blank, K25 Blank, K26 Blank, K27 Blank, K3 Blank, K32 Blank, K33 Blank, K34 Blank, K35 Blank, K36 Blank, K37 Blank, K38 Blank, K39 Blank, K4 Blank, K40 Blank, K41 Blank, K42 Blank, K43 Blank, K44 Blank, K48 Blank, K49 Blank, K5 Blank, K50 Blank, K51 Blank, K52 Blank, K53 Blank, K54 Blank, K55 Blank, K56 Blank, K57 Blank, K58 Blank, K59 Blank, K6 Blank, K60 Blank, K64 Blank, K65 Blank, K66 Blank, K67 Blank, K68 Blank, K69 Blank, K7 Blank, K70 Blank, K71 Blank, K72 Blank, K73 Blank, K74 Blank, K75 Blank, K8 Blank, K9 Blank

Commit message: Work being carried out on v2
Parts:
- added K37: Blank, Button_Switch_Keyboard:SW_Cherry_Choc5_MX_1.00u_PCB_3D, F.Cu at (203.8, 169.6)
- D0, D1, D10, D11, D16, D17, D18, D19, D2, D20, D21, D22, D23, D24, D25, D26, D27, D3, D32 (x3), D33, D34, D35, D36, D37, D38, D39, D4, D40, D41, D42, D43, D44 (x2), D48, D49, D5, D50, D51, D52, D53, D54, D55, D56, D57, D58, D59, D6, D64, D65, D66, D67, D68, D69 (x3), D7, D70 (x2), D71, D72, D73, D74, D75, D8, D9: footprint Diode_SMD:D_SOD-123 -> Stencils:Diode_THT_SOD123F_FIXED6
- K0, K1, K10, K11, K2, K3, K4, K44, K5, K6, K60, K69 (x2), K7, K70 (x2), K8, K9: footprint Button_Switch_Keyboard:SW_Cherry_MX_1.00u_PCB_HOTSWAP -> Button_Switch_Keyboard:SW_Cherry_Choc5_MX_1.00u_PCB_LED_SQUAREHOLE
- K16, K17, K18, K19, K20, K21, K22, K23, K24, K25, K26, K27, K32, K33, K34, K35, K36, K37, K38, K39, K40, K41, K42, K43, K44, K48, K49, K50, K51, K52, K53, K54, K55, K56, K57, K58, K59, K60, K64, K65, K66, K67, K68, K71, K72, K73, K74, K75: footprint Button_Switch_Keyboard:SW_Cherry_MX_1.00u_PCB_HOTSWAP -> Button_Switch_Keyboard:SW_Cherry_Choc5_MX_1.00u_PCB_3D
- moved pico 26.2 mm to (201.2, 124.4)
- moved D23 25.4 mm to (249.0, 123.1)
- moved D72 25.3 mm to (263.8, 178.2)
- moved D27 25.3 mm to (323.7, 107.5)
- moved D22 25.2 mm to (230.2, 125.2)
- moved D44 25.0 mm to (348.7, 126.2)
- moved D41 25.0 mm to (289.7, 127.4)
- moved D38 25.0 mm to (235.0, 143.6)
- moved D42 25.0 mm to (308.9, 125.4)
- moved D54 25.0 mm to (239.9, 162.0)
- moved D58 25.0 mm to (313.9, 143.8)
- moved D71 24.9 mm to (244.8, 180.5)
- moved D26 24.9 mm to (304.0, 107.0)
- moved D75 24.9 mm to (318.8, 162.2)
- moved D44 24.9 mm to (219.0, 157.8)
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Connections:
- K0 pad 2: Net-(D0-A) -> LED2
- K0 pad 3: VCC -> GND
- K0 pad 4: LED2 -> LED1
- K1 pad 2: Net-(D1-A) -> LED3
- K1 pad 3: VCC -> GND
- K1 pad 4: LED3 -> LED2
- K10 pad 2: Net-(D10-A) -> LED18
- K10 pad 3: VCC -> GND
- K10 pad 4: LED12 -> LED17
- K11 pad 3: VCC -> GND
- K11 pad 4: LED13 -> LED18
- K2 pad 2: Net-(D2-A) -> LED4
- K2 pad 3: VCC -> GND
- K2 pad 4: LED4 -> LED3
- K3 pad 2: Net-(D3-A) -> LED5
- K3 pad 3: VCC -> GND
- K3 pad 4: LED5 -> LED4
- K4 pad 2: Net-(D4-A) -> LED6
- K4 pad 3: VCC -> GND
- K4 pad 4: LED6 -> LED5
- K44 pad 2: NET-(D80-A) -> LED13
- K44 pad 3: VCC -> GND
- K44 pad 4: LED33 -> LED12
- K5 pad 2: Net-(D5-A) -> LED7
- K5 pad 3: VCC -> GND
- K5 pad 4: LED7 -> LED6
- K6 pad 2: Net-(D6-A) -> LED14
- K6 pad 3: VCC -> GND
- K6 pad 4: LED8 -> LED13
- K60 pad 2: Net-(D60-A) -> LED8
- K60 pad 3: VCC -> GND
- K60 pad 4: LED32 -> LED7
- K69 pad 2: NET-(DEXT-A) -> LED10
- K69 pad 3: VCC -> GND (x2)
- K69 pad 4: LED60 -> LED9
- K69 pad 2: Net-(D69-A) -> LED9
- K69 pad 4: LED59 -> LED8
- K7 pad 2: Net-(D7-A) -> LED15
- K7 pad 3: VCC -> GND
- K7 pad 4: LED9 -> LED14
- K70 pad 2: Net-(D61-A) -> LED11
- K70 pad 3: VCC -> GND (x2)
- K70 pad 4: LED61 -> LED10
- K70 pad 2: Net-(D70-A) -> LED12
- K70 pad 4: LED62 -> LED11
- K8 pad 2: Net-(D8-A) -> LED16
- K8 pad 3: VCC -> GND
- K8 pad 4: LED10 -> LED15
- K9 pad 2: Net-(D9-A) -> LED17
- K9 pad 3: VCC -> GND
- K9 pad 4: LED11 -> LED16
Routing:
- net VCC: track 721.2 -> 0.00 mm
- net VBUS: track 0.00 -> 560.6 mm, vias 0 -> 6
- net Row_4: track 142.2 -> 524.3 mm, vias 2 -> 0
- net Row_2: track 0.00 -> 317.2 mm
- net Row_3: track 128.1 -> 385.3 mm, vias 2 -> 0
- net Col_0: track 0.00 -> 224.5 mm
- net Row_1: track 103.5 -> 312.7 mm
- net Row_0: track 98.9 -> 305.6 mm, vias 0 -> 2
- net Col_1: track 0.00 -> 197.9 mm
- net Col_2: track 0.00 -> 178.9 mm
- net Col_3: track 0.00 -> 159.4 mm
- net Col_15: track 93.0 -> 246.2 mm, vias 5 -> 0
- net LED53: track 147.2 -> 0.00 mm
- net LED1: track 0.00 -> 146.2 mm
- net LED39: track 143.6 -> 0.00 mm
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Other:
- board text added: "Model: Ashwing66 - Rev 1.0 (Choc V1/MX) Designed by: James Gzowski (github.com/gzowski)"
- board text removed: "Model: Ashwing66 - Rev 2.0 (MX HS) Designed by: James Gzowski (github.com/gzowski)"

Commit message: Updates
Parts:
- removed the D0 at (66.3, 80.0)
- removed D1, D10, D11, D16, D17, D18, D19, D2, D20, D21, D22, D23, D24, D25, D26, D27, D3, D32 (x3), D33, D34, D35, D36, D37, D38, D39, D4, D40, D41, D42, D43, D44 (x2), D48, D49, D5, D50, D51, D52, D53, D54, D55, D56, D57, D58, D59, D6, D64, D65, D66, D67, D68, D69 (x3), D7, D70 (x2), D71, D72, D73, D74, D75, D8, D9: D, Stencils:Diode_THT_SOD123F_FIXED6
- removed G*** (x2): LOGO, LOGO
- removed the K0 at (78.1, 82.5)
- removed K1, K10, K11, K2, K3, K4, K44, K5, K6, K60, K69 (x2), K7, K70 (x2), K8, K9: Blank, Button_Switch_Keyboard:SW_Cherry_Choc5_MX_1.00u_PCB_LED_SQUAREHOLE
- removed K16, K17, K18, K19, K20, K21, K22, K23, K24, K25, K26, K27, K32, K33, K34, K35, K36, K37 (x2), K38, K39, K40, K41, K42, K43, K44, K48, K49, K50, K51, K52, K53, K54, K55, K56, K57, K58, K59, K60, K64, K65, K66, K67, K68, K71, K72, K73, K74, K75: Blank, Button_Switch_Keyboard:SW_Cherry_Choc5_MX_1.00u_PCB_3D
- removed RESET: PinHeader_1x02_P1.00mm_Vertical, Connector_PinHeader_1.00mm:PinHeader_1x02_P1.00mm_Vertical
- removed RotEnc: RotaryEncoder_EC11, Keebio-Parts:RotaryEncoder_EC11
- removed TH3 (x10): HOLE, Lily58-footprint:HOLE_M2_TH
- removed the pico at (201.2, 124.4)
- added D0: D, Stencils:Diode_THT_SOD123F_FIXED6, B.Cu at (221.8, 147.1)
- added D0: D, Stencils:Diode_THT_SOD123F_FIXED6, B.Cu at (221.8, 166.1)
- added D0: D, Stencils:Diode_THT_SOD123F_FIXED6, B.Cu at (202.8, 147.1)
- added D0: D, Stencils:Diode_THT_SOD123F_FIXED6, B.Cu at (221.8, 128.0)
- added D0: D, Stencils:Diode_THT_SOD123F_FIXED6, B.Cu at (183.7, 147.1)
- added D0: D, Stencils:Diode_THT_SOD123F_FIXED6, B.Cu at (164.7, 166.1)
- added D0: D, Stencils:Diode_THT_SOD123F_FIXED6, B.Cu at (202.8, 128.0)
- added D0: D, Stencils:Diode_THT_SOD123F_FIXED6, B.Cu at (164.7, 128.0)
- added D0: D, Stencils:Diode_THT_SOD123F_FIXED6, B.Cu at (202.8, 166.1)
- added D0: D, Stencils:Diode_THT_SOD123F_FIXED6, B.Cu at (183.7, 166.1)
- added D0: D, Stencils:Diode_THT_SOD123F_FIXED6, B.Cu at (164.7, 147.1)
- added D0: D, Stencils:Diode_THT_SOD123F_FIXED6, B.Cu at (183.7, 128.0)
- added K0: Blank, Button_Switch_Keyboard:SW_Cherry_Choc5_MX_1.00u_PCB_LED_SQUAREHOLE, F.Cu at (177.9, 161.0)
- added K0: Blank, Button_Switch_Keyboard:SW_Cherry_Choc5_MX_1.00u_PCB_LED_SQUAREHOLE, F.Cu at (216.0, 122.9)
- added K0: Blank, Button_Switch_Keyboard:SW_Cherry_Choc5_MX_1.00u_PCB_LED_SQUAREHOLE, F.Cu at (177.9, 142.0)
- added K0: Blank, Button_Switch_Keyboard:SW_Cherry_Choc5_MX_1.00u_PCB_LED_SQUAREHOLE, F.Cu at (196.9, 122.9)
- added K0: Blank, Button_Switch_Keyboard:SW_Cherry_Choc5_MX_1.00u_PCB_LED_SQUAREHOLE, F.Cu at (196.9, 142.0)
- added K0: Blank, Button_Switch_Keyboard:SW_Cherry_Choc5_MX_1.00u_PCB_LED_SQUAREHOLE, F.Cu at (158.8, 142.0)
- added K0: Blank, Button_Switch_Keyboard:SW_Cherry_Choc5_MX_1.00u_PCB_LED_SQUAREHOLE, F.Cu at (158.8, 122.9)
- added K0: Blank, Button_Switch_Keyboard:SW_Cherry_Choc5_MX_1.00u_PCB_LED_SQUAREHOLE, F.Cu at (177.9, 122.9)
- added K0: Blank, Button_Switch_Keyboard:SW_Cherry_Choc5_MX_1.00u_PCB_LED_SQUAREHOLE, F.Cu at (216.0, 161.0)
- added K0: Blank, Button_Switch_Keyboard:SW_Cherry_Choc5_MX_1.00u_PCB_LED_SQUAREHOLE, F.Cu at (216.0, 142.0)
- added K0: Blank, Button_Switch_Keyboard:SW_Cherry_Choc5_MX_1.00u_PCB_LED_SQUAREHOLE, F.Cu at (158.8, 161.0)
- added K0: Blank, Button_Switch_Keyboard:SW_Cherry_Choc5_MX_1.00u_PCB_LED_SQUAREHOLE, F.Cu at (196.9, 161.0)
- added pico: , MCU_RaspberryPi_and_Boards:RPi_Pico_SMD_TH_ALT, F.Cu at (235.3, 144.0)
Routing:
- net (no net): track 0.00 -> 1457.5 mm, vias 0 -> 4
- net VBUS: track 560.6 -> 0.00 mm, vias 6 -> 0
- net Row_4: track 524.3 -> 0.00 mm
- net Row_3: track 385.3 -> 0.00 mm
- net Row_2: track 317.2 -> 0.00 mm
- net Row_1: track 312.7 -> 0.00 mm
- net Row_0: track 305.6 -> 0.00 mm, vias 2 -> 0
- net Col_15: track 246.2 -> 0.00 mm
- net Col_0: track 224.5 -> 0.00 mm
- net Col_14: track 221.4 -> 0.00 mm
- net Col_13: track 205.6 -> 0.00 mm
- net Col_1: track 197.9 -> 0.00 mm
- net Col_12: track 190.5 -> 0.00 mm
- net Col_2: track 178.9 -> 0.00 mm
- net Col_11: track 171.4 -> 0.00 mm
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Other:
- board size 346.6 x 149.9 mm -> 100.6 x 57.4 mm
- board text removed: "BOOT"
- board text removed: "Column 01"
- board text removed: "Column 16"
- board text removed: "Model: Ashwing66 - Rev 1.0 (Choc V1/MX) Designed by: James Gzowski (github.com/gzowski)"
- board text removed: "RUN GND"
- board text removed: "Row 01"
